File: PCB/agentpad/agentpad.kicad_pcb (KiCad board)
At the start: 2 copper layers, 95 x 95 mm, 21 parts, among them J1 Conn_01x04, SW1 SW_Push, SW10 RotaryEncoder_Switch, SW2 SW_Push, SW3 SW_Push, SW4 SW_Push, SW5 SW_Push, SW6 SW_Push, SW7 SW_Push, SW8 SW_Push, SW9 SW_Push, U1 MOUDLE-SEEEDUINO-XIAO

Commit message: Re-add 6 M3 mounting holes (were deleted with LEDs); refresh gerbers.zip
The 'delete footprints with no symbols' step during LED removal also removed the
mounting holes. Re-placed H1-H6 clear of keycaps; regenerated gerbers with holes.
Parts:
- added H1: MountingHole_3.2mm_M3, MountingHole:MountingHole_3.2mm_M3, F.Cu at (65.0, 75.0)
- added H2: MountingHole_3.2mm_M3, MountingHole:MountingHole_3.2mm_M3, F.Cu at (107.5, 160.0)
- added H3: MountingHole_3.2mm_M3, MountingHole:MountingHole_3.2mm_M3, F.Cu at (65.0, 160.0)
- added H4: MountingHole_3.2mm_M3, MountingHole:MountingHole_3.2mm_M3, F.Cu at (150.0, 75.0)
- added H5: MountingHole_3.2mm_M3, MountingHole:MountingHole_3.2mm_M3, F.Cu at (150.0, 118.0)
- added H6: MountingHole_3.2mm_M3, MountingHole:MountingHole_3.2mm_M3, F.Cu at (150.0, 160.0)

Commit message: PCB: add GND pour + silkscreen branding; regenerate fab outputs
Board now has ground fill zones and 'AgentPad @znel2002' silkscreen
branding. DRC: 0 errors (27 cosmetic silk warnings only). Regenerated
gerbers.zip, board STEP, and the README PCB render.
Parts:
- moved U1 57.0 mm to (132.4, 81.6)
- moved H1 19.0 mm to (84.0, 75.0)
- moved H3 19.0 mm to (84.0, 160.0)
Routing:
- net /COL2: track 117.7 -> 69.2 mm, vias 0 -> 1
- net /COL1: track 97.4 -> 59.4 mm
- net /COL0: track 70.1 -> 97.2 mm
- net /ROW2: track 182.9 -> 158.7 mm, vias 1 -> 0
- net +3V3: track 42.9 -> 22.1 mm
- net /ENC_B: track 22.0 -> 37.9 mm
- net /OLED_SCL: track 28.8 -> 39.3 mm
- net /ROW1: track 92.5 -> 102.4 mm
- net /ENC_A: track 26.7 -> 35.9 mm
- net Net-(D9-A): track 14.6 -> 21.7 mm
- net /OLED_SDA: track 26.7 -> 33.2 mm
- net /ROW0: track 80.7 -> 86.0 mm, vias 1 -> 0
- net Net-(D4-A): track 14.7 -> 15.6 mm
- net Net-(D6-A): track 14.7 -> 15.4 mm
Other:
- board size 95 x 95 mm -> 75 x 95 mm
- board text added: "@znel2002"
- board text added: "AgentPad"
